File: hardware/versions/v1/kicad/G5FLY.kicad_sch (KiCad schematic)
At the start: 112 parts, among them IC1 MCXA154VLH, J1 SM03B-GHS-TB_LF__SN_, J10 MMCX-J-P-H-RA-TH1, J11 MMCX-J-P-H-RA-TH1, J3 USB4105-GF-A, J4 SM06B-GHS-TB_LF__SN_, J5 TagConnect_TC2030-NL, J6 SM04B-GHS-TB, J7 SM04B-GHS-TB, J8 DF40TC(2.5)-50DS-0.4V(51), J9 SM04B-GHS-TB, SW3 EVQP7J01P, U1 mosaic-G5, U10 XC8111AA01MR-G, U12 TPS7A9401DSCR, U13 XC8111AA01MR-G, U14 MP2002AGD-Z_C3751012, U2 ECMF02-2AMX6, U3 TJA1462ATK, U4 BMM350_C17225907, U6 XC8111AA01MR-G, U7 TPS7A9401DSCR, U8 MPM3632CGQV-Z, U9 XC8111AA01MR-G, Y1 OT201624MJBA4SL

Commit message: release: publish NXP hardware revision
Other:
- title: (none) -> G5Fly_NXP-MCXA154 
Changed lines of the file:
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@@
 	(generator_version "10.0")
 	(paper "A2")
+	(title_block
+		(title "G5Fly_NXP-MCXA154 ")
+		(date "2026-09-23")
+		(rev "2")
+	)
 	(rectangle
 		(start 17.78 356.87)
